File: hw/plinkyblack_hwmidi_jacks/plinkyblack_hwmidi_jacks.kicad_sch (KiCad schematic)
At the start: 283 parts, among them J1 AudioJack2_SwitchT, J1 PJ-320B, J10 AudioJack2_SwitchT, J11 AudioJack2_SwitchT, J12 Conn_02x08_Odd_Even, J13 Conn_02x08_Odd_Even, J14 AudioJack2_SwitchT, J15 AudioJack2_SwitchT, J16 AudioJack2_SwitchT, J17 AudioJack2_SwitchT, J2 AudioJack2_SwitchT, J2 PJ-320B, J20 oled0.91, J22 AudioJack2_SwitchT, J23 AudioJack2_SwitchT, J25 Conn_01x16_Female, J3 AudioJack2_SwitchT, J4 AudioJack2_SwitchT, J5 SWD header, J6 AudioJack2_SwitchT, J7 AudioJack2_SwitchT, J8 AudioJack2_SwitchT, J9 AudioJack2_SwitchT, Q1 MMBT3904, U1 HCPL-0631-500E, U1 MCP6002-xSN, U10 TL072, U11 TL072, U12 W25Q32JVSS, U13 TPS61040DBV, U14 W25Q32JVSS, U15 USBLC6-2SC6, U16 TL072, U17 LIS2DH12, U18 TL072, U19 TYPE-C-31-M-14, U2 LM1117-3.3, U20 TYPE-C-31-M-14, U3 LM1117-3.3, U4 STM32L476VGT6, U5 TL072, U6 WM8758B, U7 TL072, U8 MCP6002-xSN, U9 MCP6002-xSN, Y1 Crystal_GND24

Commit message: Removed duplicate headphone, line in and USB. Removed expansion socket.
Removed duplicate headphone, line in and USB. Removed expansion socket.
Parts:
- removed C42, C43: 220u, Capacitor_SMD:CP_Elec_6.3x5.9, symbol plinkyblack-rescue:CP-Device
- removed H1, H2, H4: MountingHole, MountingHole:MountingHole_3.2mm_M3, symbol Mechanical:MountingHole
- removed J1 (x2): PJ-320B, MyLibrary:LUOYANG-DISHANG_PJ-320B, symbol MICROMIDITRS-eagle-import:PJ-320B
- removed J25: Conn_01x16_Female, Connector_IDC:IDC-Header_2x08_P2.54mm_Horizontal, symbol plinkyblack-rescue:Conn_01x16_Female-Connector
- removed R105, R114: 5.1K, Resistor_SMD:R_0402_1005Metric, symbol Device:R
- removed R37, R56: 10k, Resistor_SMD:R_0402_1005Metric, symbol Device:R
- removed T_VBUS1: TestPoint, TestPoint:TestPoint_Pad_D1.0mm, symbol Connector:TestPoint
- removed U20: TYPE-C-31-M-14, MyLibrary:HRO_TYPE-C-31-M-12, symbol MyLibrary:TYPE-C-31-M-12
- added C10 (x2): 0.01uF, Resistor_SMD:R_0805_2012Metric, symbol Device:C_Small
- added C42, C43, C82, C83: 100uF, Capacitor_SMD:C_1206_3216Metric, symbol Device:C_Small
- added R117, R118: 10k, Resistor_SMD:R_0603_1608Metric, symbol Device:R
- FB1: value Ferrite_Bead_Small -> 600R@100MHz
- J1: Checked x -> (none); Notes (none) -> PJ366ST on Thonk
- J11: Notes (none) -> PJ398SM
- U6: value WM8758B -> WM8758CBGEFL/RV
Connections:
- net DM_C: no longer U15.1 (I/O1), U19.B7 (DN2)
- net GND: now also C10.2, C10.2
- net HPL: now also C42.1, C82.1
- net HPR: now also C43.1, C83.1
- net IO2: now also C10.1, R118.1; no longer MT1.A
- net IO3: now also C10.1, R117.1; no longer MT1.B
- net at J1.2 (TIP), R33.1: now also C42.2, C82.2
- net at J1.3 (RING), R32.1: now also C43.2, C83.2
- net DM renamed DN
- new net: MT1.A, R118.2
- new net: MT1.B, R117.2
- new net DN_C: U15.1 (I/O1), U19.B7 (DN2)
- no-connect marks 26 -> 28
Other:
- note added: "0.91 inch 128x32 I2C"
- note added: "6N137 equiv."
- note added: "ACCELEROMETER"
- note added: "KC-301249-1177582.pdf"
- note removed: "expansion header"
- note removed: "internal headers"
- title: (none) -> Plinky
- moved on the sheet: C74, D12, D23, J1, MT1, R1, R115, R116, R2, R32, R33, U15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

Commit message: Add files via upload
Parts:
- removed T_JTCK1, T_JTMS1, T_NRST1: TestPoint, TestPoint:TestPoint_Pad_D1.0mm, symbol Connector:TestPoint
- removed U19: TYPE-C-31-M-14, MyLibrary:HRO_TYPE-C-31-M-12, symbol MyLibrary:TYPE-C-31-M-12
- added J18: USB_C_Receptacle_USB2.0, Connector_USB:USB_C_Receptacle_HRO_TYPE-C-31-M-12, symbol Connector:USB_C_Receptacle_USB2.0
- C42, C43, C82, C83: LCSC (none) -> C15008; lcsc C15008 -> (none)
- R115, R116: LCSC C25779 -> C25905
- R22, R36: footprint Resistor_SMD:R_0402_1005Metric -> Resistor_SMD:R_0805_2012Metric; LCSC C25741 -> C149504
- U12, U14: footprint Package_SO:SOIC-8_5.23x5.23mm_P1.27mm -> Package_SO:SOIC-8_5.275x5.275mm_P1.27mm
- U15: Checked x -> (none); LCSC C7519 -> C2687116
Connections:
- net DN_C: now also J18.A7 (D-), J18.B7 (D-)
- net DP_C: now also J18.A6 (D+), J18.B6 (D+)
- net GND: now also R116.2, J18.A1 (GND), J18.A12 (GND), J18.B1 (GND), J18.B12 (GND), J18.S1 (SHIELD); no longer R116.1
- net VBUS: now also J18.A4 (VBUS), J18.A9 (VBUS), J18.B4 (VBUS), J18.B9 (VBUS)
- net at R115.1: now also J18.A5 (CC1)
- new net: J18.B5 (CC2), R116.1
- no-connect marks 28 -> 27
Other:
- moved on the sheet: C27, C28, C29, C31, C32, C33, C42, C43, C50, C51, C64, C74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

Commit message: Add files via upload
Parts:
- C1, C11, C16, C17, C18, C19, C2, C22, C23, C25, C28, C35, C36, C37, C40, C41, C50, C51, C52, C53, C56, C57, C58, C59, C64, C68, C69, C70, C73, C74, C77, C78: value 100n -> 100nF
- C10, C2, C26, C30, C66, C67, C71, C72, C79, C9: value 10u -> 10uF
- C10: value 0.01uF -> 10nF
- C12, C14, C15, C65: value 18p -> 18pF
- C20, C21, C75, C76: value 220p -> 220pF
- C24, C27, C29, C3, C31, C32, C33: value 4.7u -> 4.7uF
- C34, C4, C54: value 1u -> 1uF
- C38, C39, C44, C45, C46, C47, C48, C49, C5, C6, C60, C61, C62, C63, C7, C8: value 4.7n -> 4.7nF
- C55: value 10n -> 10nF
- J20: now left out of the parts list
- R1, R6, R7: value 47Ω -> 47R
- R100, R29, R38, R39, R97: value 2k2 -> 2.2k
- R117, R118: LCSC C23182 -> C25804
- R2, R94, R95, R96: value 1M5 -> 1.5M
- R2: value 15Ω -> 15R
- R3: value 470Ω -> 470R
- R4, R5: value 220Ω -> 220R
Other:
- note added: "WQP419GR or PJ366ST"
